Commit message: fix amcl param

File: linorobot2_description/urdf/robots/lino.urdf.xacro (robot description, xacro)
@@ -1,31 +1,14 @@
 <?xml version="1.0"?>
 <robot name="linorobot2_2wd" xmlns:xacro="http://ros.org/wiki/xacro">
-  <xacro:property name="base_length" value="0.34" />
-  <xacro:property name="base_width" value="0.34" />
-  <xacro:property name="base_height" value="0.07" />
-  <xacro:property name="base_mass" value="5" />
-  <xacro:property name="wheel_radius" value="0.05" />
-  <xacro:property name="wheel_width" value="0.01" />
-  <xacro:property name="wheel_pos_x" value="0.0" />
-  <xacro:property name="wheel_pos_y" value="0.175" />
-  <xacro:property name="wheel_pos_z" value="0.0" />
-  <xacro:property name="wheel_mass" value=".1" />
-  <xacro:property name="wheel_torque" value="40" />
-  <xacro:property name="front_caster_wheel" value="true" />
-  <xacro:property name="rear_caster_wheel" value="true" />
+  <xacro:arg name="sim" default="false" />
+  <xacro:include filename="$(find linorobot2_description)/urdf/lino_properties.urdf.xacro" />
   <xacro:include filename="$(find linorobot2_description)/urdf/mech/base.urdf.xacro" />
   <xacro:include filename="$(find linorobot2_description)/urdf/mech/wheel.urdf.xacro" />
   <xacro:include filename="$(find linorobot2_description)/urdf/mech/caster_wheel.urdf.xacro" />
+  <xacro:include filename="$(find linorobot2_description)/urdf/sensors/plugins.urdf.xacro" />
   <xacro:include filename="$(find linorobot2_description)/urdf/sensors/imu.urdf.xacro" />
   <xacro:include filename="$(find linorobot2_description)/urdf/sensors/generic_laser.urdf.xacro" />
   <xacro:include filename="$(find linorobot2_description)/urdf/sensors/depth_sensor.urdf.xacro" />
   <xacro:include filename="$(find linorobot2_description)/urdf/controllers/diff_drive.urdf.xacro" />
-  <xacro:property name="laser_pose">
-    <origin xyz="0.055 0.02 0.41" rpy="0 0 0"/>
-  </xacro:property>
-  <!-- Real camera z value is around 17cm, real camera x value is 13-14cm , 0.050 , 34 angle yawlidar-->
-  <xacro:property name="depth_sensor_pose">
-    <origin xyz="0.14 0.0 0.12" rpy="0 0 0"/>
-  </xacro:property>
   <xacro:base
     length="${base_length}"
@@ -35,4 +18,5 @@
     wheel_radius="${wheel_radius}"
     wheel_pos_z="${wheel_pos_z}"
+    mesh_file="${base_mesh_file}"
   />
   <xacro:wheel
@@ -44,4 +28,5 @@
     pos_z="${wheel_pos_z}"
     mass="${wheel_mass}"
+    mesh_file="${wheel_mesh_file}"
   />
   <xacro:wheel
@@ -53,4 +38,5 @@
     pos_z="${wheel_pos_z}"
     mass="${wheel_mass}"
+    mesh_file="${wheel_mesh_file}"
   />
   <xacro:if value="${front_caster_wheel}">
@@ -82,5 +68,4 @@
     wheel_separation="${wheel_pos_y * 2}"
     wheel_radius="${wheel_radius}"
-    wheel_torque="${wheel_torque}"
   />
 </robot>
