Commit message: initial added robomow_612p URDF (bo be changed a lot)

File: linorobot2_description/urdf/mech/base.urdf.xacro (robot description, xacro)
@@ -5,5 +5,5 @@
     <link name="base_link">
       <visual>
-        <origin xyz="0 0 0" rpy="0 0 0"/>
+        <origin xyz="${(length/2) - 0.1327} 0 0" rpy="0 0 0"/>
         <geometry>
           <xacro:if value="${mesh_file == ''}">
@@ -19,5 +19,5 @@
       </visual>
       <collision>
-        <origin xyz="0 0 0" rpy="0 0 0"/>
+        <origin xyz="${(length/2) - 0.0127} 0 0" rpy="0 0 0"/>
         <geometry>
           <box size="${length} ${width} ${height}"/>

File: linorobot2_description/urdf/mech/caster_wheel.urdf.xacro (robot description, xacro)
@@ -4,8 +4,8 @@
     <xacro:property name="caster_wheel_radius" value="${(wheel_radius - wheel_pos_z) / 2}" />
     <xacro:if value="${side == 'front'}">
-        <xacro:property name="caster_wheel_x" value="${(base_length / 2) - caster_wheel_radius}" />
+        <xacro:property name="caster_wheel_x" value="${base_length - caster_wheel_radius}" />
     </xacro:if>
     <xacro:if value="${side == 'rear'}">
-        <xacro:property name="caster_wheel_x" value="${-(base_length / 2) + caster_wheel_radius}" />
+        <xacro:property name="caster_wheel_x" value="${-base_length + caster_wheel_radius}" />
     </xacro:if>
     <link name="${side}_caster_wheel_link">
